Commit message: parameterised the URDF file and added tip stops

File: balanceRobot_ws/balanceRobot.urdf.xacro (robot description, xacro)
@@ -7,8 +7,9 @@
 -->
 <!-- Specify this is also an xacro extension (macro xml) -->
+<!-- Here begins the robot description with tag <robot> -->
 <robot xmlns:xacro="https://www.ros.org/wiki/xacro" name="balanceRobot">
     <!-- Material color properties -->
     <material name="gray">
-        <color rgba="0.7 0.7 0.7 1.0"/>
+        <color rgba="0.5 0.5 0.5 1.0"/>
     </material>
     <material name="red">
@@ -33,29 +34,66 @@
     </link>
     <!-- Base link stepper motors with housing -->
-    <link name="base_link"> <!-- Needs to be called base_link (as a first real link)-->
+    <!-- The dimension are defined first as parameters every dimension is in meters -->
+    <xacro:property name="HSB" value="0.083"/> <!-- HSB= Height Stepper Base (Height = x-axis) -->
+    <xacro:property name="WSB" value="0.050"/> <!-- WSB= Width Stepper Base (Width = y-axis) -->
+    <xacro:property name="LSB" value="0.046"/> <!-- LSB= Length Stepper Base (Length = z-axis) -->
+    <link name="base_link"> <!-- Needs to be called base_link (as a first real link in stead of StepperBase) -->
         <visual>
             <origin xyz="0.0 0.0 0.0" rpy="0.0 0.0 0.0"/>
             <geometry>
-                <box size="0.083 0.050 0.046"/>
+                <box size="${HSB} ${WSB} ${LSB}"/>
             </geometry>
             <material name="gray"/>
         </visual>
     </link>
-    <!-- Base Plate of the robot where everthing gets mounted -->
+    <!-- Base Plate of the robot where everthing gets mounted this geometry is approximated as a box -->
+    <!-- The dimension are defined first as parameters -->
+    <xacro:property name="HBP" value="0.083"/> <!-- HBP= Height Base Plate -->
+    <xacro:property name="WBP" value="0.108"/> <!-- WBP= Width Base Plate -->
+    <xacro:property name="LBP" value="0.007"/> <!-- LBP= Length Base Plate -->
     <link name="basePlate_link">
         <visual>
             <origin xyz="0.0 0.0 0.0" rpy="0.0 0.0 0.0"/>
             <geometry>
-                <box size="0.083 0.108 0.007"/>
+                <box size="${HBP} ${WBP} ${LBP}"/>
             </geometry>
-            <material name="red"/>
+            <material name="blue"/>
+        </visual>
+    </link>
+    <!-- Front Tip Stop of the robot (stopping the robot from tipping over to the front) -->
+    <!-- The dimension are defined first as parameters -->
+    <!-- We heavily simplify this stop as a box -->
+    <xacro:property name="HTS" value="0.020"/> <!-- HTS= Height Tip Stop -->
+    <xacro:property name="WTS" value="0.020"/> <!-- WTS= Width Tip Stop -->
+    <xacro:property name="LTS" value="0.020"/> <!-- LTS= Length Tip Stop -->
+    <link name="frontTipStop_link">
+        <visual>
+            <origin xyz="0.0 0.0 0.0" rpy="${pi*0.28} 0.0 0.0"/> <!-- turned 50 degrees on x-axis -->
+            <geometry>
+                <box size="${HTS} ${WTS} ${LTS}"/>
+            </geometry>
+            <material name="blue"/>
+        </visual>
+    </link>
+    <!-- Back Tip Stop of the robot (stopping the robot from tipping over to the back) -->
+    <link name="backTipStop_link">
+        <visual>
+            <origin xyz="0.0 0.0 0.0" rpy="-${pi*0.28} 0.0 0.0"/> <!-- turned 50 degrees on x-axis -->
+            <geometry>
+                <box size="${HTS} ${WTS} ${LTS}"/>
+            </geometry>
+            <material name="blue"/>
         </visual>
     </link>
     <!-- Main body link where battery pack and electronics are mounted -->
+    <!-- The dimension are defined first as parameters -->
+    <xacro:property name="HBL" value="0.083"/> <!-- HBL= Height Body Link -->
+    <xacro:property name="WBL" value="0.043"/> <!-- WBL= Width Body Link -->
+    <xacro:property name="LBL" value="0.170"/> <!-- LBL= Length Body Link -->
     <link name="body_link">
         <visual>
             <origin xyz="0.0 0.0 0.0" rpy="0.0 0.0 0.0"/>
             <geometry>
-                <box size="0.083 0.043 0.170"/>
+                <box size="${HBL} ${WBL} ${LBL}"/>
             </geometry>
             <material name="white"/>
@@ -63,19 +101,25 @@
     </link>
     <!-- Top Plate link the platform on top of the robot -->
+    <!-- The dimension are defined first as parameters -->
+    <xacro:property name="RTP" value="0.054"/> <!-- RPB= Radius Top Plate -->
+    <xacro:property name="LTP" value="0.007"/> <!-- LPB= Length Top Plate -->
     <link name="topPlate_link">
         <visual>
             <origin xyz="0.0 0.0 0.0" rpy="0.0 0.0 0.0"/>
             <geometry>
-                <cylinder radius="0.054" length="0.007"/>
+                <cylinder radius="${RTP}" length="${LTP}"/>
             </geometry>
-            <material name="red"/>
+            <material name="blue"/>
         </visual>
     </link>
     <!-- Link that represents the right wheel-->
+    <!-- The dimension are defined first as parameters -->
+    <xacro:property name="RW" value="0.0375"/> <!-- RW= Radius Wheel -->
+    <xacro:property name="LW" value="0.024"/> <!-- LW= Length Wheel -->
     <link name="right_wheel_link">
         <visual>
             <origin xyz="0.0 0.0 0.0" rpy="0.0 ${pi/2} 0.0"/>
             <geometry>
-                <cylinder radius="0.0375" length="0.024"/>
+                <cylinder radius="${RW}" length="${LW}"/>
             </geometry>
             <material name="black"/>
@@ -87,5 +131,5 @@
             <origin xyz="0.0 0.0 0.0" rpy="0.0 ${pi/2} 0.0"/>
             <geometry>
-                <cylinder radius="0.0375" length="0.024"/>
+                <cylinder radius="${RW}" length="${LW}"/>
             </geometry>
             <material name="black"/>
@@ -94,6 +138,7 @@
     <!-- Joints of the robot they attach the links together to make a TF tree -->
     <!-- Joint that connects the virtual base_footprint and base_link -->
+    <!-- This link makes sure the origin is on the ground in the middle of the robot-->
     <joint name="base_footprint_joint" type="fixed">
-        <origin xyz="0.0 0.0 0.0375" rpy="0.0 0.0 0.0"/>
+        <origin xyz="0.0 0.0 ${RW}" rpy="0.0 0.0 0.0"/> <!-- Offset is the radius of a (right) wheel -->
         <parent link="base_footprint"/>
         <child link="base_link"/>
@@ -101,11 +146,23 @@
     <!-- Joint that connects base_link with baseplate -->
     <joint name="base_plate_joint" type="fixed">
-        <origin xyz="0.0 0.0 0.0265" rpy="0.0 0.0 0.0"/>
+        <origin xyz="0.0 0.0 ${(LSB/2) + (LBP/2)}" rpy="0.0 0.0 0.0"/> <!-- half-LSB+half-LBP (0.023+0.0035)=0.0265-->
         <parent link="base_link"/>
         <child link="basePlate_link"/>
     </joint>
+    <!-- Joint that connects the frontTipStop with the baseplate -->
+    <joint name="plate_ftip_joint" type="fixed">
+        <origin xyz="0.0 -${(WBP/2)} -${(LTS/2) + (LBP/2)}" rpy="0.0 0.0 0.0"/>
+        <parent link="basePlate_link"/>
+        <child link="frontTipStop_link"/>
+    </joint>
+    <!-- Joint that connects the frontTipStop with the baseplate -->
+    <joint name="plate_btip_joint" type="fixed">
+        <origin xyz="0.0 ${(WBP/2)} -${(LTS/2) + (LBP/2)}" rpy="0.0 0.0 0.0"/>
+        <parent link="basePlate_link"/>
+        <child link="backTipStop_link"/>
+    </joint>
     <!-- Joint that links the main body with respect to the base_link -->
     <joint name="base_body_link" type="fixed">
-        <origin xyz="0.0 0.0 0.115" rpy="0.0 0.0 0.0"/>
+        <origin xyz="0.0 0.0 ${(LSB/2) + LBP + (LBL/2)}" rpy="0.0 0.0 0.0"/> <!-- half-LSB+LBP+half-LBL (0.023+0.007+0.085)=0.115 -->
         <parent link="base_link"/>
         <child link="body_link"/>
@@ -113,21 +170,23 @@
     <!-- Joint that links the top plate with respect to the base_link -->
     <joint name="base_topPlate_joint" type="fixed">
-        <origin xyz="0.0 0.0 0.2035" rpy="0.0 0.0 0.0"/>
+        <origin xyz="0.0 0.0 ${(LSB/2) + LBP + LBL + (LTP/2)}" rpy="0.0 0.0 0.0"/> <!-- Half-LSB+LBP+LBL+half-LTP (0.023+0.007+0.17+0.0035=0.2035)-->
         <parent link="base_link"/>
         <child link="topPlate_link"/>
     </joint>
     <!-- Joint that links the right wheel to the base_link as a continous rotating wheel -->
+    <!-- Outside dimensions of wheels measure 137,50mm of the real robot -->
+    <xacro:property name="ODW" value="0.1375"/> <!-- ODW= Outside dimension wheels-->
     <joint name="right_wheel_joint" type="continuous">
-        <origin xyz="0.0555 0.0 0.0" rpy="0.0 0.0 0.0"/>
+        <origin xyz="${(ODW/2)-(LW/2)} 0.0 0.0" rpy="0.0 0.0 0.0"/> <!-- 0.1375/2-0.024/2=0.05675 -->
         <parent link="base_link"/>
         <child link="right_wheel_link"/>
-        <axis xyz="1.0 0.0 0.0"/>
+        <axis xyz="1.0 0.0 0.0"/> <!-- continuous rotation is around the x-axis -->
     </joint>
     <!-- Joint that links the left wheel to the base_link as a continous rotating wheel -->
     <joint name="left_wheel_joint" type="continuous">
-        <origin xyz="-0.0555 0.0 0.0" rpy="0.0 0.0 0.0"/>
+        <origin xyz="-${(ODW/2)-(LW/2)} 0.0 0.0" rpy="0.0 0.0 0.0"/>
         <parent link="base_link"/>
         <child link="left_wheel_link"/>
-        <axis xyz="1.0 0.0 0.0"/> <!-- Let the wheel rotate around the x-axis -->
+        <axis xyz="1.0 0.0 0.0"/> <!-- continuous rotation is around the x-axis -->
     </joint>
 </robot>
