Commit message: added collision tags to the URDF file

File: balanceRobot_ws/src/balance_robot/robot_description/balanceRobot.urdf.xacro (robot description, xacro)
@@ -46,4 +46,10 @@
             <material name="gray"/>
         </visual>
+        <collision>
+            <origin xyz="0.0 0.0 0.0" rpy="0.0 0.0 0.0"/>
+            <geometry>
+                <box size="${HSB} ${WSB} ${LSB}"/>
+            </geometry>
+        </collision>
     </link>
     <!-- Base Plate of the robot where everthing gets mounted this geometry is approximated as a box -->
@@ -60,4 +66,10 @@
             <material name="blue"/>
         </visual>
+        <collision>
+            <origin xyz="0.0 0.0 0.0" rpy="0.0 0.0 0.0"/>
+            <geometry>
+                <box size="${HBP} ${WBP} ${LBP}"/>
+            </geometry>
+        </collision>
     </link>
     <!-- Front Tip Stop of the robot (stopping the robot from tipping over to the front) -->
@@ -75,4 +87,10 @@
             <material name="blue"/>
         </visual>
+        <collision>
+            <origin xyz="0.0 0.0 0.0" rpy="${pi*0.28} 0.0 0.0"/>
+            <geometry>
+                <box size="${HTS} ${WTS} ${LTS}"/>
+            </geometry>
+        </collision>
     </link>
     <!-- Back Tip Stop of the robot (stopping the robot from tipping over to the back) -->
@@ -85,4 +103,10 @@
             <material name="blue"/>
         </visual>
+        <collision>
+            <origin xyz="0.0 0.0 0.0" rpy="-${pi*0.28} 0.0 0.0"/>
+            <geometry>
+                <box size="${HTS} ${WTS} ${LTS}"/>
+            </geometry>
+        </collision>
     </link>
     <!-- Main body link where battery pack and electronics are mounted -->
@@ -99,4 +123,10 @@
             <material name="white"/>
         </visual>
+        <collision>
+            <origin xyz="0.0 0.0 0.0" rpy="0.0 0.0 0.0"/>
+            <geometry>
+                <box size="${HBL} ${WBL} ${LBL}"/>
+            </geometry>
+        </collision>
     </link>
     <!-- Top Plate link the platform on top of the robot -->
@@ -112,4 +142,10 @@
             <material name="blue"/>
         </visual>
+        <collision>
+            <origin xyz="0.0 0.0 0.0" rpy="0.0 0.0 0.0"/>
+            <geometry>
+                <cylinder radius="${RTP}" length="${LTP}"/>
+            </geometry>
+        </collision>
     </link>
     <!-- Link that represents the right wheel-->
@@ -125,4 +161,10 @@
             <material name="black"/>
         </visual>
+        <collision>
+            <origin xyz="0.0 0.0 0.0" rpy="0.0 ${pi/2} 0.0"/>
+            <geometry>
+                <cylinder radius="${RW}" length="${LW}"/>
+            </geometry>
+        </collision>
     </link>
     <!-- Link that represents the left wheel -->
@@ -135,4 +177,10 @@
             <material name="black"/>
         </visual>
+        <collision>
+            <origin xyz="0.0 0.0 0.0" rpy="0.0 ${pi/2} 0.0"/>
+            <geometry>
+                <cylinder radius="${RW}" length="${LW}"/>
+            </geometry>
+        </collision>
     </link>
     <!-- Joints of the robot they attach the links together to make a TF tree -->

Commit message: Added visual meshes to the URDF file

File: balanceRobot_ws/src/balance_robot/robot_description/balanceRobot.urdf.xacro (robot description, xacro)
@@ -42,7 +42,8 @@
             <origin xyz="0.0 0.0 0.0" rpy="0.0 0.0 0.0"/>
             <geometry>
-                <box size="${HSB} ${WSB} ${LSB}"/>
-            </geometry>
-            <material name="gray"/>
+                <!-- <box size="${HSB} ${WSB} ${LSB}"/> -->
+                <mesh filename="package://balance_robot/meshes/StepperBase.dae"/>
+            </geometry>
+            <!-- <material name="gray"/> -->
         </visual>
         <collision>
@@ -62,7 +63,8 @@
             <origin xyz="0.0 0.0 0.0" rpy="0.0 0.0 0.0"/>
             <geometry>
-                <box size="${HBP} ${WBP} ${LBP}"/>
-            </geometry>
-            <material name="blue"/>
+                <!-- <box size="${HBP} ${WBP} ${LBP}"/> -->
+                <!-- <mesh filename="package://balance_robot/meshes/BasePlate.dae"/> -->
+            </geometry>
+            <!-- <material name="blue"/> -->
         </visual>
         <collision>
@@ -81,9 +83,10 @@
     <link name="frontTipStop_link">
         <visual>
-            <origin xyz="0.0 0.0 0.0" rpy="${pi*0.28} 0.0 0.0"/> <!-- turned 50 degrees on x-axis -->
-            <geometry>
-                <box size="${HTS} ${WTS} ${LTS}"/>
-            </geometry>
-            <material name="blue"/>
+            <origin xyz="0.0 0.0065 0.0" rpy="${(pi*0.28)+(pi/2)} 0.0 ${pi}"/> <!-- turned 50 degrees on x-axis -->
+            <geometry>
+                <!-- <box size="${HTS} ${WTS} ${LTS}"/> -->
+                <mesh filename="package://balance_robot/meshes/TipOverStop.dae"/>
+            </geometry>
+            <!-- <material name="blue"/> -->
         </visual>
         <collision>
@@ -97,9 +100,10 @@
     <link name="backTipStop_link">
         <visual>
-            <origin xyz="0.0 0.0 0.0" rpy="-${pi*0.28} 0.0 0.0"/> <!-- turned 50 degrees on x-axis -->
-            <geometry>
-                <box size="${HTS} ${WTS} ${LTS}"/>
-            </geometry>
-            <material name="blue"/>
+            <origin xyz="0.0 -0.0065 0.0" rpy="${(pi*0.28)-(1.5*pi)} 0.0 0.0"/> <!-- turned 50 degrees on x-axis -->
+            <geometry>
+                <!-- <box size="${HTS} ${WTS} ${LTS}"/> -->
+                <mesh filename="package://balance_robot/meshes/TipOverStop.dae"/>
+            </geometry>
+            <!-- <material name="blue"/> -->
         </visual>
         <collision>
@@ -114,12 +118,13 @@
     <xacro:property name="HBL" value="0.083"/> <!-- HBL= Height Body Link -->
     <xacro:property name="WBL" value="0.043"/> <!-- WBL= Width Body Link -->
-    <xacro:property name="LBL" value="0.170"/> <!-- LBL= Length Body Link -->
+    <xacro:property name="LBL" value="0.150"/> <!-- LBL= Length Body Link -->
     <link name="body_link">
         <visual>
-            <origin xyz="0.0 0.0 0.0" rpy="0.0 0.0 0.0"/>
-            <geometry>
-                <box size="${HBL} ${WBL} ${LBL}"/>
-            </geometry>
-            <material name="white"/>
+            <origin xyz="0.00045 0.0 -0.0135" rpy="0.0 0.0 0.0"/>
+            <geometry>
+                <!-- <box size="${HBL} ${WBL} ${LBL}"/> -->
+                <mesh filename="package://balance_robot/meshes/MainBody.dae"/>
+            </geometry>
+            <!-- <material name="white"/> -->
         </visual>
         <collision>
@@ -136,9 +141,10 @@
     <link name="topPlate_link">
         <visual>
-            <origin xyz="0.0 0.0 0.0" rpy="0.0 0.0 0.0"/>
-            <geometry>
-                <cylinder radius="${RTP}" length="${LTP}"/>
-            </geometry>
-            <material name="blue"/>
+            <origin xyz="0.0001 -0.0015 0.0" rpy="0.0 0.0 0.0"/>
+            <geometry>
+                <!-- <cylinder radius="${RTP}" length="${LTP}"/> -->
+                <mesh filename="package://balance_robot/meshes/TopPlate.dae"/>
+            </geometry>
+            <!-- <material name="blue"/> -->
         </visual>
         <collision>
@@ -155,9 +161,10 @@
     <link name="right_wheel_link">
         <visual>
-            <origin xyz="0.0 0.0 0.0" rpy="0.0 ${pi/2} 0.0"/>
-            <geometry>
-                <cylinder radius="${RW}" length="${LW}"/>
-            </geometry>
-            <material name="black"/>
+            <origin xyz="0.0 0.0 0.0" rpy="0.0 0.0 0.0"/>
+            <geometry>
+                <!-- <cylinder radius="${RW}" length="${LW}"/> -->
+                <mesh filename="package://balance_robot/meshes/Wheel.dae"/>
+            </geometry>
+            <!-- <material name="black"/> -->
         </visual>
         <collision>
@@ -171,9 +178,10 @@
     <link name="left_wheel_link">
         <visual>
-            <origin xyz="0.0 0.0 0.0" rpy="0.0 ${pi/2} 0.0"/>
-            <geometry>
-                <cylinder radius="${RW}" length="${LW}"/>
-            </geometry>
-            <material name="black"/>
+            <origin xyz="0.0 0.0 0.0" rpy="0.0 0.0 0.0"/>
+            <geometry>
+                <!-- <cylinder radius="${RW}" length="${LW}"/> -->
+                <mesh filename="package://balance_robot/meshes/Wheel.dae"/>
+            </geometry>
+            <!-- <material name="black"/> -->
         </visual>
         <collision>
@@ -226,5 +234,5 @@
     <xacro:property name="ODW" value="0.1375"/> <!-- ODW= Outside dimension wheels-->
     <joint name="right_wheel_joint" type="continuous">
-        <origin xyz="${(ODW/2)-(LW/2)} 0.0 0.0" rpy="0.0 0.0 0.0"/> <!-- 0.1375/2-0.024/2=0.05675 -->
+        <origin xyz="${(ODW/2)-(LW/2)} 0.0 -0.001" rpy="0.0 0.0 0.0"/> <!-- 0.1375/2-0.024/2=0.05675 -->
         <parent link="base_link"/>
         <child link="right_wheel_link"/>
@@ -233,5 +241,5 @@
     <!-- Joint that links the left wheel to the base_link as a continous rotating wheel -->
     <joint name="left_wheel_joint" type="continuous">
-        <origin xyz="-${(ODW/2)-(LW/2)} 0.0 0.0" rpy="0.0 0.0 0.0"/>
+        <origin xyz="-${(ODW/2)-(LW/2)} 0.0 -0.001" rpy="0.0 0.0 0.0"/>
         <parent link="base_link"/>
         <child link="left_wheel_link"/>
