Commit message: Added sim launch file

File: balanceRobot_ws/src/balance_robot/robot_description/balance_robot.urdf.xacro (robot description, xacro)
@@ -11,4 +11,6 @@
     <!-- Include xacro files -->
     <xacro:include filename="inertial_macros.xacro"/>
+    <!-- Put on meshes -->
+    <xacro:arg name="use_meshes" default="false"/>
     <!-- Material color properties -->
     <material name="gray">
@@ -46,6 +48,10 @@
             <origin xyz="0.0 0.0 0.0" rpy="0.0 0.0 0.0"/>
             <geometry>
-                <!-- <box size="${HSB} ${WSB} ${LSB}"/> -->
-                <mesh filename="package://balance_robot/robot_description/meshes/StepperBase.dae"/>
+                <xacro:if value="$(arg use_meshes)">
+                    <mesh filename="package://balance_robot/robot_description/meshes/StepperBase.dae"/>
+                </xacro:if>
+                <xacro:unless value="$(arg use_meshes)">
+                    <box size="${HSB} ${WSB} ${LSB}"/>
+                </xacro:unless>
             </geometry>
             <material name="gray"/>
@@ -95,6 +101,10 @@
             <origin xyz="0.0 0.0065 0.0" rpy="${(pi*0.28)+(pi/2)} 0.0 ${pi}"/> <!-- turned 50 degrees on x-axis -->
             <geometry>
-                <!-- <box size="${HTS} ${WTS} ${LTS}"/> -->
-                <mesh filename="package://balance_robot/robot_description/meshes/TipOverStop.dae"/>
+                <xacro:if value="$(arg use_meshes)">
+                    <mesh filename="package://balance_robot/robot_description/meshes/TipOverStop.dae"/>
+                </xacro:if>
+                <xacro:unless value="$(arg use_meshes)">
+                    <box size="${HTS} ${WTS} ${LTS}"/>
+                </xacro:unless>
             </geometry>
             <material name="blue"/>
@@ -115,6 +125,10 @@
             <origin xyz="0.0 -0.0065 0.0" rpy="${(pi*0.28)-(1.5*pi)} 0.0 0.0"/> <!-- turned 50 degrees on x-axis -->
             <geometry>
-                <!-- <box size="${HTS} ${WTS} ${LTS}"/> -->
-                <mesh filename="package://balance_robot/robot_description/meshes/TipOverStop.dae"/>
+                <xacro:if value="$(arg use_meshes)">
+                    <mesh filename="package://balance_robot/robot_description/meshes/TipOverStop.dae"/>
+                </xacro:if>
+                <xacro:unless value="$(arg use_meshes)">
+                    <box size="${HTS} ${WTS} ${LTS}"/>
+                </xacro:unless>
             </geometry>
             <material name="blue"/>
@@ -139,6 +153,10 @@
             <origin xyz="0.00045 0.0 -0.0135" rpy="0.0 0.0 0.0"/>
             <geometry>
-                <!-- <box size="${HBL} ${WBL} ${LBL}"/> -->
-                <mesh filename="package://balance_robot/robot_description/meshes/MainBody.dae"/>
+                <xacro:if value="$(arg use_meshes)">
+                    <mesh filename="package://balance_robot/robot_description/meshes/MainBody.dae"/>
+                </xacro:if>
+                <xacro:unless value="$(arg use_meshes)">
+                    <box size="${HBL} ${WBL} ${LBL}"/>
+                </xacro:unless>
             </geometry>
             <material name="white"/>
@@ -164,6 +182,10 @@
             <origin xyz="0.0 -0.0075 -0.005" rpy="0.0 0.0 0.0"/>
             <geometry>
-                <!-- <box size="${HBPL} ${WBPL} ${LBPL}"/> -->
-                <mesh filename="package://balance_robot/robot_description/meshes/PowerBank.dae"/>
+                <xacro:if value="$(arg use_meshes)">
+                    <mesh filename="package://balance_robot/robot_description/meshes/PowerBank.dae"/>
+                </xacro:if>
+                <xacro:unless value="$(arg use_meshes)">
+                    <box size="${HBPL} ${WBPL} ${LBPL}"/>
+                </xacro:unless>
             </geometry>
             <material name="green"/>
@@ -187,6 +209,10 @@
             <origin xyz="0.0001 -0.0015 0.0" rpy="0.0 0.0 0.0"/>
             <geometry>
-                <!-- <cylinder radius="${RTP}" length="${LTP}"/> -->
-                <mesh filename="package://balance_robot/robot_description/meshes/TopPlate.dae"/>
+                <xacro:if value="$(arg use_meshes)">
+                    <mesh filename="package://balance_robot/robot_description/meshes/TopPlate.dae"/>
+                </xacro:if>
+                <xacro:unless value="$(arg use_meshes)">
+                    <cylinder radius="${RTP}" length="${LTP}"/>
+                </xacro:unless>
             </geometry>
             <material name="blue"/>
@@ -207,10 +233,15 @@
     <xacro:property name="RW" value="0.0375"/> <!-- RW= Radius Wheel -->
     <xacro:property name="LW" value="0.024"/> <!-- LW= Length Wheel -->
+    <xacro:property name="LWM" value="0.040"/> <!-- LWM= Left Wheel Mass-->
     <link name="right_wheel_link">
         <visual>
-            <origin xyz="0.0 0.0 0.0" rpy="0.0 0.0 0.0"/>
-            <geometry>
-                <!-- <cylinder radius="${RW}" length="${LW}"/> -->
-                <mesh filename="package://balance_robot/robot_description/meshes/Wheel.dae"/>
+            <origin xyz="0.0 0.0 0.0" rpy="0.0 ${pi/2} 0.0"/>
+            <geometry>
+                <xacro:if value="$(arg use_meshes)">
+                    <mesh filename="package://balance_robot/robot_description/meshes/Wheel.dae"/>
+                </xacro:if>
+                <xacro:unless value="$(arg use_meshes)">
+                    <cylinder radius="${RW}" length="${LW}"/>
+                </xacro:unless>
             </geometry>
             <material name="black"/>
@@ -229,8 +260,12 @@
     <link name="left_wheel_link">
         <visual>
-            <origin xyz="0.0 0.0 0.0" rpy="0.0 0.0 0.0"/>
-            <geometry>
-                <!-- <cylinder radius="${RW}" length="${LW}"/> -->
-                <mesh filename="package://balance_robot/robot_description/meshes/Wheel.dae"/>
+            <origin xyz="0.0 0.0 0.0" rpy="0.0 ${pi/2} 0.0"/>
+            <geometry>
+                <xacro:if value="$(arg use_meshes)">
+                    <mesh filename="package://balance_robot/robot_description/meshes/Wheel.dae"/>
+                </xacro:if>
+                <xacro:unless value="$(arg use_meshes)">
+                    <cylinder radius="${RW}" length="${LW}"/>
+                </xacro:unless>
             </geometry>
             <material name="black"/>
@@ -242,7 +277,21 @@
             </geometry>
         </collision>
+        <inertial>
+            <origin xyz="0.0 0.0 0.0" rpy="${pi/2} 0.0 0.0"/>
+            <mass value="${LWM}"/>
+            <inertia ixx="${(LWM/12)*(3*RW*RW+LW*LW)}" ixy="0.0" ixz="0.0" iyy="${(LWM/12)*(3*RW*RW+LW*LW)}" iyz="0.0" izz="${(LWM/2)*(RW*RW)}"/>
+        </inertial>
+        <!--
+        <xacro:macro name="cylinder_inertia" params="mass r h">
+        <intertial>
+            <origin xyz="0.0 0.0 0.0" rpy="0.0 ${pi/2} 0.0"/>
+            <mass value="${mass}"/>
+            <inertia ixx="${(mass/12)*(3*r*r+h*h)}" ixy="0.0" ixz="0.0" iyy="${(mass/12)*(3*r*r+h*h)}" iyz="0.0" izz="${(mass/2)*(r*r)}"/>
+        </intertial>
+        </xacro:macro>
         <xacro:inertial_cylinder mass="0.040" length="${LW}" radius="${RW}">
             <origin xyz="0.0 0.0 0.0" rpy="0.0 ${pi/2} 0.0"/>
         </xacro:inertial_cylinder>
+        -->
     </link>
     <!-- Joints of the robot they attach the links together to make a TF tree -->
@@ -306,3 +355,17 @@
         <axis xyz="1.0 0.0 0.0"/> <!-- continuous rotation is around the x-axis -->
     </joint>
+    <gazebo reference="right_wheel_link">
+        <material>Gazebo/Black</material>
+    </gazebo>
+    <gazebo reference="left_wheel_link">
+        <material>Gazebo/Black</material>
+    </gazebo>
+    <!-- Gazebo specific code ... -->
+    <gazebo>
+        <plugin name="gazebo_ros_joint_state_publisher" filename="libgazebo_ros_joint_state_publisher.so">
+            <update_rate>20</update_rate> <!-- Update rate is equal to 20 Hz-->
+            <joint_name>right_wheel_joint</joint_name>
+            <joint_name>left_wheel_joint</joint_name>
+        </plugin>
+    </gazebo>
 </robot>

Commit message: fixed origins/inertias and simulation

File: balanceRobot_ws/src/balance_robot/robot_description/balance_robot.urdf.xacro (robot description, xacro)
@@ -44,4 +44,5 @@
     <xacro:property name="WSB" value="0.050"/> <!-- WSB= Width Stepper Base (Width = y-axis) -->
     <xacro:property name="LSB" value="0.046"/> <!-- LSB= Length Stepper Base (Length = z-axis) -->
+    <xacro:property name="MSB" value="0.622"/> <!-- MSB= Mass Stepper Base -->
     <link name="base_link"> <!-- Needs to be called base_link (as a first real link in stead of StepperBase) -->
         <visual>
@@ -63,5 +64,5 @@
             </geometry>
         </collision>
-        <xacro:inertial_box mass="0.622" x="${HSB}" y="${WSB}" z="${LSB}">
+        <xacro:inertial_box mass="${MSB}" x="${HSB}" y="${WSB}" z="${LSB}">
             <origin xyz="0.0 0.0 0.0" rpy="0.0 0.0 0.0"/>
         </xacro:inertial_box>
@@ -69,7 +70,8 @@
     <!-- Base Plate of the robot where everthing gets mounted this geometry is approximated as a box -->
     <!-- The dimensions are defined first as parameters -->
-    <xacro:property name="HBP" value="0.083"/> <!-- HBP= Height Base Plate -->
-    <xacro:property name="WBP" value="0.108"/> <!-- WBP= Width Base Plate -->
-    <xacro:property name="LBP" value="0.007"/> <!-- LBP= Length Base Plate -->
+    <xacro:property name="HBP" value="0.083"/> <!-- HBP= Height Base Plate (Height = x-axis) -->
+    <xacro:property name="WBP" value="0.108"/> <!-- WBP= Width Base Plate (Width = y-axis) -->
+    <xacro:property name="LBP" value="0.007"/> <!-- LBP= Length Base Plate (Length = z-axis) -->
+    <xacro:property name="MBP" value="0.050"/> <!-- MBP= Mass Base Plate -->
     <link name="basePlate_link">
         <visual>
@@ -87,5 +89,5 @@
             </geometry>
         </collision>
-        <xacro:inertial_box mass="0.050" x="${HBP}" y="${WBP}" z="${LBP}">
+        <xacro:inertial_box mass="${MBP}" x="${HBP}" y="${WBP}" z="${LBP}">
             <origin xyz="0.0 0.0 0.0" rpy="0.0 0.0 0.0"/>
         </xacro:inertial_box>
@@ -94,10 +96,11 @@
     <!-- The dimensions are defined first as parameters -->
     <!-- We heavily simplify this stop as a box -->
-    <xacro:property name="HTS" value="0.020"/> <!-- HTS= Height Tip Stop -->
-    <xacro:property name="WTS" value="0.020"/> <!-- WTS= Width Tip Stop -->
-    <xacro:property name="LTS" value="0.020"/> <!-- LTS= Length Tip Stop -->
+    <xacro:property name="HTS" value="0.020"/> <!-- HTS= Height Tip Stop (Height = x-axis) -->
+    <xacro:property name="WTS" value="0.020"/> <!-- WTS= Width Tip Stop (Width = y-axis) -->
+    <xacro:property name="LTS" value="0.020"/> <!-- LTS= Length Tip Stop (Length = z-axis) -->
+    <xacro:property name="MTS" value="0.020"/> <!-- MTS= Mass Tip Stop -->
     <link name="frontTipStop_link">
         <visual>
-            <origin xyz="0.0 0.0065 0.0" rpy="${(pi*0.28)+(pi/2)} 0.0 ${pi}"/> <!-- turned 50 degrees on x-axis -->
+            <origin xyz="0.0 0.0065 0.0" rpy="0.0 0.0 0.0"/> <!-- turned 50 degrees on x-axis -->
             <geometry>
                 <xacro:if value="$(arg use_meshes)">
@@ -111,10 +114,10 @@
         </visual>
         <collision>
-            <origin xyz="0.0 0.0065 0.0" rpy="-${(pi*0.28)} 0.0 0.0"/>
+            <origin xyz="0.0 0.0065 0.0" rpy="0.0 0.0 0.0"/>
             <geometry>
                 <box size="${HTS} ${WTS} ${LTS}"/>
             </geometry>
         </collision>
-        <xacro:inertial_box mass="0.020" x="${HTS}" y="${WTS}" z="${LTS}">
+        <xacro:inertial_box mass="${MTS}" x="${HTS}" y="${WTS}" z="${LTS}">
             <origin xyz="0.0 0.0065 0.0" rpy="-${(pi*0.28)} 0.0 0.0"/>
         </xacro:inertial_box>
@@ -123,5 +126,5 @@
     <link name="backTipStop_link">
         <visual>
-            <origin xyz="0.0 -0.0065 0.0" rpy="${(pi*0.28)-(1.5*pi)} 0.0 0.0"/> <!-- turned 50 degrees on x-axis -->
+            <origin xyz="0.0 -0.0065 0.0" rpy="0.0 0.0 0.0"/> <!-- turned 50 degrees on x-axis -->
             <geometry>
                 <xacro:if value="$(arg use_meshes)">
@@ -135,18 +138,19 @@
         </visual>
         <collision>
+            <origin xyz="0.0 -0.0065 0.0" rpy="0.0 0.0 0.0"/>
+            <geometry>
+                <box size="${HTS} ${WTS} ${LTS}"/>
+            </geometry>
+        </collision>
+        <xacro:inertial_box mass="${MTS}" x="${HTS}" y="${WTS}" z="${LTS}">
             <origin xyz="0.0 -0.0065 0.0" rpy="${(pi*0.28)-(1.5*pi)} 0.0 0.0"/>
-            <geometry>
-                <box size="${HTS} ${WTS} ${LTS}"/>
-            </geometry>
-        </collision>
-        <xacro:inertial_box mass="0.020" x="${HTS}" y="${WTS}" z="${LTS}">
-            <origin xyz="0.0 -0.0065 0.0" rpy="${(pi*0.28)-(1.5*pi)} 0.0 0.0"/>
         </xacro:inertial_box>
     </link>
     <!-- Main body link where battery pack and electronics are mounted -->
     <!-- The dimensions are defined first as parameters -->
-    <xacro:property name="HBL" value="0.083"/> <!-- HBL= Height Body Link -->
-    <xacro:property name="WBL" value="0.043"/> <!-- WBL= Width Body Link -->
-    <xacro:property name="LBL" value="0.150"/> <!-- LBL= Length Body Link -->
+    <xacro:property name="HBL" value="0.083"/> <!-- HBL= Height Body Link (Height = x-axis) -->
+    <xacro:property name="WBL" value="0.043"/> <!-- WBL= Width Body Link (Width = y-axis) -->
+    <xacro:property name="LBL" value="0.150"/> <!-- LBL= Length Body Link (Length = z-axis) -->
+    <xacro:property name="MBL" value="0.127"/> <!-- MBL= Mass Body Link -->
     <link name="body_link">
         <visual>
@@ -168,5 +172,5 @@
             </geometry>
         </collision>
-        <xacro:inertial_box mass="0.127" x="${HBL}" y="${WBL}" z="${LBL}">
+        <xacro:inertial_box mass="${MBL}" x="${HBL}" y="${WBL}" z="${LBL}">
             <origin xyz="0.0 0.0 0.0" rpy="0.0 0.0 0.0"/>
         </xacro:inertial_box>
@@ -175,7 +179,8 @@
     <!-- a significant influence on the dynamic behaviour -->
     <!-- The dimensions are defined first as parameters -->
-    <xacro:property name="HBPL" value="0.087"/> <!-- HBP= Height Battery Pack Link -->
-    <xacro:property name="WBPL" value="0.026"/> <!-- WBP= Width Battery Pack Link -->
-    <xacro:property name="LBPL" value="0.0936"/> <!-- LBP= Length Battery Pack Link -->
+    <xacro:property name="HBPL" value="0.087"/> <!-- HBPL= Height Battery Pack Link (Height = x-axis) -->
+    <xacro:property name="WBPL" value="0.026"/> <!-- WBPL= Width Battery Pack Link (Width = y-axis) -->
+    <xacro:property name="LBPL" value="0.0936"/> <!-- LBPL= Length Battery Pack Link (Length = z-axis) -->
+    <xacro:property name="MBPL" value="0.265"/> <!-- MBPL= Mass Battery Pack Link -->
     <link name="batteryPack_link">
         <visual>
@@ -197,5 +202,5 @@
             </geometry>
         </collision>
-        <xacro:inertial_box mass="0.265" x="${HBPL}" y="${WBPL}" z="${LBPL}">
+        <xacro:inertial_box mass="${MBPL}" x="${HBPL}" y="${WBPL}" z="${LBPL}">
             <origin xyz="0.0 0.0 -0.005" rpy="0.0 0.0 0.0"/>
         </xacro:inertial_box>
@@ -203,6 +208,7 @@
     <!-- Top Plate link the platform on top of the robot -->
     <!-- The dimensions are defined first as parameters -->
-    <xacro:property name="RTP" value="0.054"/> <!-- RPB= Radius Top Plate -->
-    <xacro:property name="LTP" value="0.007"/> <!-- LPB= Length Top Plate -->
+    <xacro:property name="RTP" value="0.054"/> <!-- RPB= Radius Top Plate (Radius = x,y-axis) -->
+    <xacro:property name="LTP" value="0.007"/> <!-- LPB= Length Top Plate (Length = z-axis) -->
+    <xacro:property name="MTP" value="0.059"/> <!-- MTP= Mass Top Plate -->
     <link name="topPlate_link">
         <visual>
@@ -224,5 +230,5 @@
             </geometry>
         </collision>
-        <xacro:inertial_cylinder mass="0.059" length="${LTP}" radius="${RTP}">
+        <xacro:inertial_cylinder mass="${MTP}" length="${LTP}" radius="${RTP}">
             <origin xyz="0.0 0.0 0.0" rpy="0.0 0.0 0.0"/>
         </xacro:inertial_cylinder>
@@ -231,10 +237,10 @@
     <!-- Link that represents the right wheel-->
     <!-- The dimensions are defined first as parameters -->
-    <xacro:property name="RW" value="0.0375"/> <!-- RW= Radius Wheel -->
-    <xacro:property name="LW" value="0.024"/> <!-- LW= Length Wheel -->
-    <xacro:property name="LWM" value="0.040"/> <!-- LWM= Left Wheel Mass-->
+    <xacro:property name="RW" value="0.0375"/> <!-- RW= Radius Wheel (Radius = x,y-axis) -->
+    <xacro:property name="LW" value="0.024"/> <!-- LW= Length Wheel (Length = z-axis) -->
+    <xacro:property name="MW" value="0.040"/> <!-- MW= Mass Wheel -->
     <link name="right_wheel_link">
         <visual>
-            <origin xyz="0.0 0.0 0.0" rpy="0.0 ${pi/2} 0.0"/>
+            <origin xyz="0.0 0.0 0.0" rpy="0.0 0.0 0.0"/>
             <geometry>
                 <xacro:if value="$(arg use_meshes)">
@@ -248,11 +254,11 @@
         </visual>
         <collision>
-            <origin xyz="0.0 0.0 0.0" rpy="0.0 ${pi/2} 0.0"/>
+            <origin xyz="0.0 0.0 0.0" rpy="0.0 0.0 0.0"/>
             <geometry>
                 <cylinder radius="${RW}" length="${LW}"/>
             </geometry>
         </collision>
-        <xacro:inertial_cylinder mass="0.040" length="${LW}" radius="${RW}">
-            <origin xyz="0.0 0.0 0.0" rpy="0.0 ${pi/2} 0.0"/>
+        <xacro:inertial_cylinder mass="${MW}" length="${LW}" radius="${RW}">
+            <origin xyz="0.0 0.0 0.0" rpy="0.0 0.0 0.0"/>
         </xacro:inertial_cylinder>
     </link>
@@ -260,5 +266,5 @@
     <link name="left_wheel_link">
         <visual>
-            <origin xyz="0.0 0.0 0.0" rpy="0.0 ${pi/2} 0.0"/>
+            <origin xyz="0.0 0.0 0.0" rpy="0.0 0.0 0.0"/>
             <geometry>
                 <xacro:if value="$(arg use_meshes)">
@@ -272,14 +278,12 @@
         </visual>
         <collision>
-            <origin xyz="0.0 0.0 0.0" rpy="0.0 ${pi/2} 0.0"/>
+            <origin xyz="0.0 0.0 0.0" rpy="0.0 0.0 0.0"/>
             <geometry>
                 <cylinder radius="${RW}" length="${LW}"/>
             </geometry>
         </collision>
-        <inertial>
-            <origin xyz="0.0 0.0 0.0" rpy="${pi/2} 0.0 0.0"/>
-            <mass value="${LWM}"/>
-            <inertia ixx="${(LWM/12)*(3*RW*RW+LW*LW)}" ixy="0.0" ixz="0.0" iyy="${(LWM/12)*(3*RW*RW+LW*LW)}" iyz="0.0" izz="${(LWM/2)*(RW*RW)}"/>
-        </inertial>
+        <xacro:inertial_cylinder mass="${MW}" length="${LW}" radius="${RW}">
+            <origin xyz="0.0 0.0 0.0" rpy="0.0 0.0 0.0"/>
+        </xacro:inertial_cylinder>
         <!--
         <xacro:macro name="cylinder_inertia" params="mass r h">
@@ -290,7 +294,9 @@
         </intertial>
         </xacro:macro>
-        <xacro:inertial_cylinder mass="0.040" length="${LW}" radius="${RW}">
-            <origin xyz="0.0 0.0 0.0" rpy="0.0 ${pi/2} 0.0"/>
-        </xacro:inertial_cylinder>
+        <inertial>
+            <origin xyz="0.0 0.0 0.0" rpy="0.0 0.0 0.0"/>
+            <mass value="${MW}"/>
+            <inertia ixx="${(MW/12)*(3*RW*RW+LW*LW)}" ixy="0.0" ixz="0.0" iyy="${(MW/12)*(3*RW*RW+LW*LW)}" iyz="0.0" izz="${(MW/2)*(RW*RW)}"/>
+        </inertial>
         -->
     </link>
@@ -311,11 +317,11 @@
     <!-- Joint that connects the frontTipStop with the baseplate -->
     <joint name="plate_ftip_joint" type="fixed">
-        <origin xyz="0.0 -${(WBP/2)} -${(LTS/2) + (LBP/2)}" rpy="0.0 0.0 0.0"/>
+        <origin xyz="0.0 -${(WBP/2)} -${(LTS/2) + (LBP/2)}" rpy="${(pi*0.28)} 0.0 0.0"/>
         <parent link="basePlate_link"/>
         <child link="frontTipStop_link"/>
     </joint>
-    <!-- Joint that connects the frontTipStop with the baseplate -->
+    <!-- Joint that connects the backTipStop with the baseplate -->
     <joint name="plate_btip_joint" type="fixed">
-        <origin xyz="0.0 ${(WBP/2)} -${(LTS/2) + (LBP/2)}" rpy="0.0 0.0 0.0"/>
+        <origin xyz="0.0 ${(WBP/2)} -${(LTS/2) + (LBP/2)}" rpy="-${(pi*0.28)} 0.0 0.0"/>
         <parent link="basePlate_link"/>
         <child link="backTipStop_link"/>
@@ -343,16 +349,39 @@
     <xacro:property name="ODW" value="0.1375"/> <!-- ODW= Outside dimension wheels-->
     <joint name="right_wheel_joint" type="continuous">
-        <origin xyz="${(ODW/2)-(LW/2)} 0.0 -0.001" rpy="0.0 0.0 0.0"/> <!-- 0.1375/2-0.024/2=0.05675 -->
+        <origin xyz="${(ODW/2)-(LW/2)} 0.0 -0.001" rpy="0.0 ${pi/2} 0.0"/> <!-- 0.1375/2-0.024/2=0.05675 -->
         <parent link="base_link"/>
         <child link="right_wheel_link"/>
-        <axis xyz="1.0 0.0 0.0"/> <!-- continuous rotation is around the x-axis -->
+        <axis xyz="0.0 0.0 1.0"/> <!-- continuous rotation is around the z-axis -->
     </joint>
     <!-- Joint that links the left wheel to the base_link as a continous rotating wheel -->
     <joint name="left_wheel_joint" type="continuous">
-        <origin xyz="-${(ODW/2)-(LW/2)} 0.0 -0.001" rpy="0.0 0.0 0.0"/>
+        <origin xyz="-${(ODW/2)-(LW/2)} 0.0 -0.001" rpy="0.0 ${pi/2} 0.0"/>
         <parent link="base_link"/>
         <child link="left_wheel_link"/>
-        <axis xyz="1.0 0.0 0.0"/> <!-- continuous rotation is around the x-axis -->
-    </joint>
+        <axis xyz="0.0 0.0 1.0"/> <!-- continuous rotation is around the z-axis -->
+    </joint>
+    <!-- Gazebo specific code ... -->
+    <!-- Set the Gazebo colors -->
+    <gazebo reference="base_link">
+        <material>Gazebo/Gray</material>
+    </gazebo>
+    <gazebo reference="basePlate_link">
+        <material>Gazebo/Blue</material>
+    </gazebo>
+    <gazebo reference="frontTipStop_link">
+        <material>Gazebo/Blue</material>
+    </gazebo>
+    <gazebo reference="backTipStop_link">
+        <material>Gazebo/Blue</material>
+    </gazebo>
+    <gazebo reference="body_link">
+        <material>Gazebo/White</material>
+    </gazebo>
+    <gazebo reference="batteryPack_link">
+        <material>Gazebo/Green</material>
+    </gazebo>
+    <gazebo reference="topPlate_link">
+        <material>Gazebo/Blue</material>
+    </gazebo>
     <gazebo reference="right_wheel_link">
         <material>Gazebo/Black</material>
@@ -361,5 +390,4 @@
         <material>Gazebo/Black</material>
     </gazebo>
-    <!-- Gazebo specific code ... -->
     <gazebo>
         <plugin name="gazebo_ros_joint_state_publisher" filename="libgazebo_ros_joint_state_publisher.so">
