Commit message: Added IMU sensor and start rviz in launch file

File: balanceRobot_ws/src/balance_robot/robot_description/balance_robot.urdf.xacro (robot description, xacro)
@@ -2,4 +2,5 @@
 <robot xmlns:xacro="https://www.ros.org/wiki/xacro" name="balance_robot">
    <xacro:include filename="balance_robot_core.xacro"/>
+   <xacro:include filename="IMU_sensor.xacro"/>
    <xacro:include filename="gazebo_control.xacro"/>
 </robot>

File: balanceRobot_ws/src/balance_robot/robot_description/balance_robot_core.xacro (robot description, xacro)
@@ -13,4 +13,5 @@
     <!-- Put on meshes -->
     <xacro:arg name="use_meshes" default="true"/>
+    <xacro:arg name='use_footprint' default="false"/>
     <!-- Material color properties -->
     <material name="gray">
@@ -35,7 +36,9 @@
     <!-- Links of the robot they describe the (objects/parts) of the robot -->
     <!-- Link that is on the ground in the middle of the robot (useful for navigation purposes -->
-    <link name="base_footprint"> <!-- Conventional name for this virtual reference link -->
-        <!-- Empty virtual link-->
-    </link>
+    <xacro:if value="$(arg use_footprint)">
+        <link name="base_footprint"> <!-- Conventional name for this virtual reference link -->
+            <!-- Empty virtual link-->
+        </link>
+    </xacro:if>
     <!-- ********************** ROBOT BASE *********************************  -->
     <!-- Base link stepper motors with housing -->
@@ -102,5 +105,5 @@
     <link name="frontTipStop_link">
         <visual>
-            <origin xyz="0.0 0.0065 0.0" rpy="0.0 0.0 0.0"/> <!-- turned 50 degrees on x-axis -->
+            <origin xyz="0.0 0.001 -0.0075" rpy="${pi + (0.06*pi)} 0.0 ${pi}"/> <!-- turned 50 degrees on x-axis -->
             <geometry>
                 <xacro:if value="$(arg use_meshes)">
@@ -126,5 +129,5 @@
     <link name="backTipStop_link">
         <visual>
-            <origin xyz="0.0 -0.0065 0.0" rpy="0.0 0.0 0.0"/> <!-- turned 50 degrees on x-axis -->
+            <origin xyz="0.0 -0.001 -0.0075" rpy="${pi + (0.06*pi)} 0.0 0.0"/> <!-- turned 50 degrees on x-axis -->
             <geometry>
                 <xacro:if value="$(arg use_meshes)">
@@ -175,4 +178,18 @@
             <origin xyz="0.0 0.0 0.0" rpy="0.0 0.0 0.0"/>
         </xacro:inertial_box>
+    </link>
+    <!-- IMU link that is where the IMU is located -->
+    <!-- The dimensions are defined first as parameters -->
+    <xacro:property name="HIL" value="0.0025"/> <!-- HIL= Height IMU Link (Height = x-axis) -->
+    <xacro:property name="WIL" value="0.001"/> <!-- WIL= Width IMU Link (Width = y-axis) -->
+    <xacro:property name="LIL" value="0.003"/> <!-- LIL= Length IMU Link (Length = z-axis) -->
+    <link name="imu_link">
+        <visual>
+            <origin xyz="0.0 0.0 0.0" rpy="0.0 0.0 0.0"/>
+            <geometry>
+                <box size="${HIL} ${WIL} ${LIL}"/>
+            </geometry>
+            <material name="black"/>
+        </visual>
     </link>
     <!-- Battery pack link, this is taken as a separate link because the inertia and mass have -->
@@ -300,9 +317,11 @@
     <!-- Joint that connects the virtual base_footprint and base_link -->
     <!-- This link makes sure the origin is on the ground in the middle of the robot-->
-    <joint name="base_footprint_joint" type="fixed">
-        <origin xyz="0.0 0.0 ${RW}" rpy="0.0 0.0 0.0"/> <!-- Offset is the radius of a (right) wheel -->
-        <parent link="base_footprint"/>
-        <child link="base_link"/>
-    </joint>
+    <xacro:if value="$(arg use_footprint)">
+        <joint name="base_footprint_joint" type="fixed">
+            <origin xyz="0.0 0.0 ${RW}" rpy="0.0 0.0 0.0"/> <!-- Offset is the radius of a (right) wheel -->
+            <parent link="base_footprint"/>
+            <child link="base_link"/>
+        </joint>
+    </xacro:if>
     <!-- Joint that connects base_link with baseplate -->
     <joint name="base_plate_joint" type="fixed">
@@ -328,4 +347,10 @@
         <parent link="base_link"/>
         <child link="body_link"/>
+    </joint>
+    <!-- Joint that links the IMU sensor to the main body -->
+    <joint name="body_imu_joint" type="fixed">
+        <origin xyz="0.010 -0.03 0.015" rpy="0.0 0.0 0.0"/>
+        <parent link="body_link"/>
+        <child link="imu_link"/>
     </joint>
     <!-- Joint that links the battery pack to the main body -->

Commit message: added some thing on ubuntu

File: balanceRobot_ws/src/balance_robot/robot_description/balance_robot.urdf.xacro (robot description, xacro)
@@ -1,22 +1,19 @@
 <?xml version="1.0"?> <!-- Specify this is an xml file using version 1.0-->
 <robot xmlns:xacro="https://www.ros.org/wiki/xacro" name="balance_robot">
-   <!-- Parameters
-   <xacro:arg name="use_ros2_control" default="true"/>
- -->
+   <!-- URDF custom parameters -->
+   <xacro:arg name="use_meshes" default="true"/> <!-- Put on meshes -->
+   <xacro:arg name='use_footprint' default="false"/> <!-- Use footpriny link -->
+   <xacro:arg name="use_ros2_control" default="false"/> <!-- Use ros2_control -->
    <!-- This file includes the core of the robot -->
    <xacro:include filename="balance_robot_core.xacro"/>
    <!-- Simulating a IMU sensor -->
    <xacro:include filename="IMU_sensor.xacro"/>
-   <xacro:include filename="ros2_control.xacro"/>
    <!-- Use ros2_control -->
-   <!--
-   <xacro:if value="$(use_ros2_control)">
+   <xacro:if value="$(arg use_ros2_control)">
+      <xacro:include filename="ros2_control.xacro"/>
    </xacro:if>
-   -->
    <!-- Use build in Gazebo control -->
-   <!--
-   <xacro:unless value="$(use_ros2_control)">
+   <xacro:unless value="$(arg use_ros2_control)">
       <xacro:include filename="gazebo_control.xacro"/>
    </xacro:unless>
-   -->
 </robot>

File: balanceRobot_ws/src/balance_robot/robot_description/balance_robot_core.xacro (robot description, xacro)
@@ -11,7 +11,4 @@
     <!-- Include xacro files -->
     <xacro:include filename="inertial_macros.xacro"/>
-    <!-- Put on meshes -->
-    <xacro:arg name="use_meshes" default="true"/>
-    <xacro:arg name='use_footprint' default="false"/>
     <!-- Material color properties -->
     <material name="gray">
@@ -81,6 +78,10 @@
             <origin xyz="0.0 0.0 0.0" rpy="0.0 0.0 0.0"/>
             <geometry>
-                <box size="${HBP} ${WBP} ${LBP}"/>
-                <!-- <mesh filename="package://balance_robot/robot_description/meshes/BasePlate.dae"/> -->
+                <xacro:if value="$(arg use_meshes)">
+                    <mesh filename="package://balance_robot/meshes/BasePlate.dae"/>
+                </xacro:if>
+                <xacro:unless value="$(arg use_meshes)">
+                    <box size="${HBP} ${WBP} ${LBP}"/>
+                </xacro:unless>
             </geometry>
             <material name="blue"/>
@@ -161,5 +162,5 @@
             <geometry>
                 <xacro:if value="$(arg use_meshes)">
-                    <mesh filename="package://balance_robot/meshes/MainBody.dae"/>
+                    <mesh filename="package://balance_robot/meshes/MainBodyColor.dae"/>
                 </xacro:if>
                 <xacro:unless value="$(arg use_meshes)">
@@ -267,5 +268,5 @@
             <geometry>
                 <xacro:if value="$(arg use_meshes)">
-                    <mesh filename="package://balance_robot/meshes/Wheel.dae"/>
+                    <mesh filename="package://balance_robot/meshes/WheelColor.dae"/>
                 </xacro:if>
                 <xacro:unless value="$(arg use_meshes)">
@@ -296,5 +297,5 @@
             <geometry>
                 <xacro:if value="$(arg use_meshes)">
-                    <mesh filename="package://balance_robot/meshes/Wheel.dae"/>
+                    <mesh filename="package://balance_robot/meshes/WheelColor.dae"/>
                 </xacro:if>
                 <xacro:unless value="$(arg use_meshes)">

Commit message: updated launch file and URDF file

File: balanceRobot_ws/src/balance_robot/robot_description/balance_robot.urdf.xacro (robot description, xacro)
@@ -5,4 +5,5 @@
    <xacro:arg name='use_footprint' default="false"/> <!-- Use footpriny link -->
    <xacro:arg name="use_ros2_control" default="false"/> <!-- Use ros2_control -->
+   <xacro:arg name="use_gazebo_colors" default="false"/> <!-- Use Gazebo collors -->
    <!-- This file includes the core of the robot -->
    <xacro:include filename="balance_robot_core.xacro"/>

File: balanceRobot_ws/src/balance_robot/robot_description/balance_robot_core.xacro (robot description, xacro)
@@ -385,36 +385,44 @@
     <!-- Gazebo specific code ... -->
     <!-- Set the Gazebo colors -->
-    <gazebo reference="base_link">
-        <material>Gazebo/Gray</material>
-    </gazebo>
-    <gazebo reference="basePlate_link">
-        <material>Gazebo/Blue</material>
-    </gazebo>
+    <xacro:if value="$(arg use_gazebo_colors)">
+        <gazebo reference="base_link">
+            <material>Gazebo/Gray</material>
+        </gazebo>
+        <gazebo reference="basePlate_link">
+            <material>Gazebo/Blue</material>
+        </gazebo>
+    </xacro:if>
     <!-- Make the Tip Over Stops have some amount of friction with respect to the ground -->
     <gazebo reference="frontTipStop_link">
-        <material>Gazebo/Blue</material>
+        <xacro:if value="$(arg use_gazebo_colors)">
+            <material>Gazebo/Blue</material>
+        </xacro:if>
         <mu1 value="0.5"/>
         <mu2 value="0.5"/>
     </gazebo>
     <gazebo reference="backTipStop_link">
-        <material>Gazebo/Blue</material>
+        <xacro:if value="$(arg use_gazebo_colors)">
+            <material>Gazebo/Blue</material>
+        </xacro:if>
         <mu1 value="0.5"/>
         <mu2 value="0.5"/>
     </gazebo>
-    <gazebo reference="body_link">
-        <material>Gazebo/White</material>
-    </gazebo>
-    <gazebo reference="batteryPack_link">
-        <material>Gazebo/Gray</material>
-    </gazebo>
-    <gazebo reference="topPlate_link">
-        <material>Gazebo/Blue</material>
-    </gazebo>
-    <gazebo reference="right_wheel_link">
-        <material>Gazebo/Black</material>
-    </gazebo>
-    <gazebo reference="left_wheel_link">
-        <material>Gazebo/Black</material>
-    </gazebo>
+    <xacro:if value="$(arg use_gazebo_colors)">
+        <gazebo reference="body_link">
+            <material>Gazebo/White</material>
+        </gazebo>
+        <gazebo reference="batteryPack_link">
+            <material>Gazebo/Gray</material>
+        </gazebo>
+        <gazebo reference="topPlate_link">
+            <material>Gazebo/Blue</material>
+        </gazebo>
+        <gazebo reference="right_wheel_link">
+            <material>Gazebo/Black</material>
+        </gazebo>
+        <gazebo reference="left_wheel_link">
+            <material>Gazebo/Black</material>
+        </gazebo>
+    </xacro:if>
     <!-- Gazebo requires the use of plugins to interact with other systems such as ROS2 -->
     <!-- This plugin will publish the joint_states for the selected joints
@@ -427,4 +435,3 @@
         </plugin>
     </gazebo>
-    <!-- *********************** IMU SETUP *********************************  -->
 </robot>
