Commit message: fixed Gazebo mesh visualization

File: balanceRobot_ws/src/balance_robot/robot_description/balance_robot_core.xacro (robot description, xacro)
@@ -12,5 +12,5 @@
     <xacro:include filename="inertial_macros.xacro"/>
     <!-- Put on meshes -->
-    <xacro:arg name="use_meshes" default="false"/>
+    <xacro:arg name="use_meshes" default="true"/>
     <!-- Material color properties -->
     <material name="gray">
@@ -50,5 +50,5 @@
             <geometry>
                 <xacro:if value="$(arg use_meshes)">
-                    <mesh filename="package://balance_robot/robot_description/meshes/StepperBase.dae"/>
+                    <mesh filename="package://balance_robot/meshes/StepperBase.dae"/>
                 </xacro:if>
                 <xacro:unless value="$(arg use_meshes)">
@@ -105,5 +105,5 @@
             <geometry>
                 <xacro:if value="$(arg use_meshes)">
-                    <mesh filename="package://balance_robot/robot_description/meshes/TipOverStop.dae"/>
+                    <mesh filename="package://balance_robot/meshes/TipOverStop.dae"/>
                 </xacro:if>
                 <xacro:unless value="$(arg use_meshes)">
@@ -129,5 +129,5 @@
             <geometry>
                 <xacro:if value="$(arg use_meshes)">
-                    <mesh filename="package://balance_robot/robot_description/meshes/TipOverStop.dae"/>
+                    <mesh filename="package://balance_robot/meshes/TipOverStop.dae"/>
                 </xacro:if>
                 <xacro:unless value="$(arg use_meshes)">
@@ -158,5 +158,5 @@
             <geometry>
                 <xacro:if value="$(arg use_meshes)">
-                    <mesh filename="package://balance_robot/robot_description/meshes/MainBody.dae"/>
+                    <mesh filename="package://balance_robot/meshes/MainBody.dae"/>
                 </xacro:if>
                 <xacro:unless value="$(arg use_meshes)">
@@ -188,5 +188,5 @@
             <geometry>
                 <xacro:if value="$(arg use_meshes)">
-                    <mesh filename="package://balance_robot/robot_description/meshes/PowerBank.dae"/>
+                    <mesh filename="package://balance_robot/meshes/PowerBank.dae"/>
                 </xacro:if>
                 <xacro:unless value="$(arg use_meshes)">
@@ -216,5 +216,5 @@
             <geometry>
                 <xacro:if value="$(arg use_meshes)">
-                    <mesh filename="package://balance_robot/robot_description/meshes/TopPlate.dae"/>
+                    <mesh filename="package://balance_robot/meshes/TopPlate.dae"/>
                 </xacro:if>
                 <xacro:unless value="$(arg use_meshes)">
@@ -250,5 +250,5 @@
             <geometry>
                 <xacro:if value="$(arg use_meshes)">
-                    <mesh filename="package://balance_robot/robot_description/meshes/Wheel.dae"/>
+                    <mesh filename="package://balance_robot/meshes/Wheel.dae"/>
                 </xacro:if>
                 <xacro:unless value="$(arg use_meshes)">
@@ -279,5 +279,5 @@
             <geometry>
                 <xacro:if value="$(arg use_meshes)">
-                    <mesh filename="package://balance_robot/robot_description/meshes/Wheel.dae"/>
+                    <mesh filename="package://balance_robot/meshes/Wheel.dae"/>
                 </xacro:if>
                 <xacro:unless value="$(arg use_meshes)">
@@ -368,6 +368,6 @@
     <gazebo reference="frontTipStop_link">
         <material>Gazebo/Blue</material>
-        <mu1 value="1"/>
-        <mu2 value="1"/>
+        <mu1 value="0.5"/>
+        <mu2 value="0.5"/>
     </gazebo>
     <gazebo reference="backTipStop_link">
@@ -380,5 +380,5 @@
     </gazebo>
     <gazebo reference="batteryPack_link">
-        <material>Gazebo/Green</material>
+        <material>Gazebo/Gray</material>
     </gazebo>
     <gazebo reference="topPlate_link">

Commit message: finished the simulation with all meshes and Gazebo control plugin

File: balanceRobot_ws/src/balance_robot/robot_description/balance_robot_core.xacro (robot description, xacro)
@@ -50,5 +50,5 @@
             <geometry>
                 <xacro:if value="$(arg use_meshes)">
-                    <mesh filename="package://balance_robot/meshes/StepperBase.dae"/>
+                    <mesh filename="package://balance_robot/meshes/StepperBaseV1Color.dae"/>
                 </xacro:if>
                 <xacro:unless value="$(arg use_meshes)">
@@ -106,8 +106,8 @@
     <link name="frontTipStop_link">
         <visual>
-            <origin xyz="0.0 0.001 -0.0075" rpy="${pi + (0.06*pi)} 0.0 ${pi}"/> <!-- turned 50 degrees on x-axis -->
-            <geometry>
-                <xacro:if value="$(arg use_meshes)">
-                    <mesh filename="package://balance_robot/meshes/TipOverStop.dae"/>
+            <origin xyz="0.0 0.005 -0.004" rpy="${pi + (0.03*pi)} 0.0 ${pi}"/> <!-- turned 50 degrees on x-axis -->
+            <geometry>
+                <xacro:if value="$(arg use_meshes)">
+                    <mesh filename="package://balance_robot/meshes/TipOverStopColor.dae"/>
                 </xacro:if>
                 <xacro:unless value="$(arg use_meshes)">
@@ -130,8 +130,8 @@
     <link name="backTipStop_link">
         <visual>
-            <origin xyz="0.0 -0.001 -0.0075" rpy="${pi + (0.06*pi)} 0.0 0.0"/> <!-- turned 50 degrees on x-axis -->
-            <geometry>
-                <xacro:if value="$(arg use_meshes)">
-                    <mesh filename="package://balance_robot/meshes/TipOverStop.dae"/>
+            <origin xyz="0.0 -0.005 -0.004" rpy="${pi + (0.03*pi)} 0.0 0.0"/> <!-- turned 50 degrees on x-axis -->
+            <geometry>
+                <xacro:if value="$(arg use_meshes)">
+                    <mesh filename="package://balance_robot/meshes/TipOverStopColor.dae"/>
                 </xacro:if>
                 <xacro:unless value="$(arg use_meshes)">
@@ -162,5 +162,5 @@
             <geometry>
                 <xacro:if value="$(arg use_meshes)">
-                    <mesh filename="package://balance_robot/meshes/MainBodyColor.dae"/>
+                    <mesh filename="package://balance_robot/meshes/MainBodyV1Color.dae"/>
                 </xacro:if>
                 <xacro:unless value="$(arg use_meshes)">
@@ -206,5 +206,5 @@
             <geometry>
                 <xacro:if value="$(arg use_meshes)">
-                    <mesh filename="package://balance_robot/meshes/PowerBank.dae"/>
+                    <mesh filename="package://balance_robot/meshes/PowerBankColor.dae"/>
                 </xacro:if>
                 <xacro:unless value="$(arg use_meshes)">
@@ -234,5 +234,5 @@
             <geometry>
                 <xacro:if value="$(arg use_meshes)">
-                    <mesh filename="package://balance_robot/meshes/TopPlate.dae"/>
+                    <mesh filename="package://balance_robot/meshes/TopPlateColor.dae"/>
                 </xacro:if>
                 <xacro:unless value="$(arg use_meshes)">
@@ -315,4 +315,5 @@
         </xacro:inertial_cylinder>
     </link>
+    <xacro:property name="Z_OFFZ" value="0.002"/>
     <!-- Joints of the robot they attach the links together to make a TF tree -->
     <!-- Joint that connects the virtual base_footprint and base_link -->
@@ -327,5 +328,5 @@
     <!-- Joint that connects base_link with baseplate -->
     <joint name="base_plate_joint" type="fixed">
-        <origin xyz="0.0 0.0 ${(LSB/2) + (LBP/2)}" rpy="0.0 0.0 0.0"/> <!-- half-LSB+half-LBP (0.023+0.0035)=0.0265-->
+        <origin xyz="0.0 0.0 ${(LSB/2) + (LBP/2)-Z_OFFZ}" rpy="0.0 0.0 0.0"/> <!-- half-LSB+half-LBP (0.023+0.0035)=0.0265-->
         <parent link="base_link"/>
         <child link="basePlate_link"/>
@@ -333,5 +334,5 @@
     <!-- Joint that connects the frontTipStop with the baseplate -->
     <joint name="plate_ftip_joint" type="fixed">
-        <origin xyz="0.0 -${(WBP/2)} -${(LTS/2) + (LBP/2)}" rpy="${(pi*0.28)} 0.0 0.0"/>
+        <origin xyz="0.0 -${(WBP/2)} -0.015" rpy="${(pi*0.25)} 0.0 0.0"/>
         <parent link="basePlate_link"/>
         <child link="frontTipStop_link"/>
@@ -339,5 +340,5 @@
     <!-- Joint that connects the backTipStop with the baseplate -->
     <joint name="plate_btip_joint" type="fixed">
-        <origin xyz="0.0 ${(WBP/2)} -${(LTS/2) + (LBP/2)}" rpy="-${(pi*0.28)} 0.0 0.0"/>
+        <origin xyz="0.0 ${(WBP/2)} -0.015" rpy="-${(pi*0.25)} 0.0 0.0"/>
         <parent link="basePlate_link"/>
         <child link="backTipStop_link"/>
@@ -345,5 +346,5 @@
     <!-- Joint that links the main body with respect to the base_link -->
     <joint name="base_body_joint" type="fixed">
-        <origin xyz="0.0 0.0 ${(LSB/2) + LBP + (LBL/2)}" rpy="0.0 0.0 0.0"/> <!-- half-LSB+LBP+half-LBL (0.023+0.007+0.085)=0.115 -->
+        <origin xyz="0.0 0.0 ${(LSB/2) + LBP + (LBL/2)-0.001-Z_OFFZ}" rpy="0.0 0.0 0.0"/> <!-- half-LSB+LBP+half-LBL (0.023+0.007+0.085)=0.115 -->
         <parent link="base_link"/>
         <child link="body_link"/>
@@ -363,5 +364,5 @@
     <!-- Joint that links the top plate with respect to the base_link -->
     <joint name="base_topPlate_joint" type="fixed">
-        <origin xyz="0.0 0.0 ${(LSB/2) + LBP + LBL + (LTP/2)}" rpy="0.0 0.0 0.0"/> <!-- Half-LSB+LBP+LBL+half-LTP (0.023+0.007+0.17+0.0035=0.2035)-->
+        <origin xyz="0.0 0.0 ${(LSB/2) + LBP + LBL + (LTP/2)-0.0035}" rpy="0.0 0.0 0.0"/> <!-- Half-LSB+LBP+LBL+half-LTP (0.023+0.007+0.17+0.0035=0.2035)-->
         <parent link="base_link"/>
         <child link="topPlate_link"/>
